File: PCB/LLatmega128_e_paper_9_1.kicad_sch (KiCad schematic)
At the start: 23 parts, among them J1 AVR-ISP-6, J2 Conn_01x06_Male, J3 ePaper, J4 Conn_02x14_Counter_Clockwise, Q1 PN2222A, SW1 SW_Push, SW2 SW_Push, SW3 SW_Push, SW4 SW_Push, U1 ATmega128-16A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

Commit message: edit & update
Other:
- moved on the sheet: BZ1, Q1, R7
