File: PCB/LLatmega128_e_paper_9_1_emver.kicad_pcb (KiCad board)
At the start: 2 copper layers, 67 x 63 mm, 37 parts, among them J1 AVR-ISP-6, J2 Conn_01x06_Male, J3 ePaper, J4 Conn_02x14_Counter_Clockwise, Q1 PN2222A, SW1 SW_Push, SW2 SW_Push, SW3 SW_Push, SW4 SW_Push, U1 ATmega128-16A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

Commit message: edit & update
Routing:
- net /RST: track 55.0 -> 54.3 mm
- net GND: vias 108 -> 122
